Commit message: nav added

File: src_gazebo/urdf/src_body.urdf (robot description, URDF)
Before this commit: robot src_body, 10 links, 9 joints
Links:
- link base_link: geometry collision mesh filename=/home/kimsooyoung/ros2_ws/install/src_gazebo/share/src_gaze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 scale=0.001 0.001 0.001; visual mesh filename=/home/kimsooyoung/ros2_ws/install/src_gazebo/share/src_gaze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 scale=0.001 0.001 0.001
- link lf_wheel_link: geometry collision mesh filename=/home/kimsooyoung/ros2_ws/install/src_gazebo/share/src_gaze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 scale=0.001 0.001 0.001; visual mesh filename=/home/kimsooyoung/ros2_ws/install/src_gazebo/share/src_gaze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 scale=0.001 0.001 0.001
- link logi_camera_link: geometry collision mesh filename=/home/kimsooyoung/ros2_ws/install/src_gazebo/share/src_gaze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 scale=0.001 0.001 0.001; visual mesh filename=/home/kimsooyoung/ros2_ws/install/src_gazebo/share/src_gaze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 scale=0.001 0.001 0.001
- link lr_wheel_link: geometry collision mesh filename=/home/kimsooyoung/ros2_ws/install/src_gazebo/share/src_gaze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 scale=0.001 0.001 0.001; visual mesh filename=/home/kimsooyoung/ros2_ws/install/src_gazebo/share/src_gaze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 scale=0.001 0.001 0.001
- link rf_wheel_link: geometry collision mesh filename=/home/kimsooyoung/ros2_ws/install/src_gazebo/share/src_gaze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 scale=0.001 0.001 0.001; visual mesh filename=/home/kimsooyoung/ros2_ws/install/src_gazebo/share/src_gaze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 scale=0.001 0.001 0.001
- link rplidar_a2_link: geometry collision mesh filename=/home/kimsooyoung/ros2_ws/install/src_gazebo/share/src_gaze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 scale=0.001 0.001 0.001; visual mesh filename=/home/kimsooyoung/ros2_ws/install/src_gazebo/share/src_gaze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 scale=0.001 0.001 0.001
- link rr_wheel_link: geometry collision mesh filename=/home/kimsooyoung/ros2_ws/install/src_gazebo/share/src_gaze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 scale=0.001 0.001 0.001; visual mesh filename=/home/kimsooyoung/ros2_ws/install/src_gazebo/share/src_gaze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 scale=0.001 0.001 0.001
