Commit message: base footprint added - urdf

File: src_gazebo/urdf/src_body.urdf.xacro (robot description, xacro)
@@ -5,4 +5,5 @@
   <xacro:include filename="$(find src_gazebo)/urdf/src_body.gazebo" />
   <!-- <xacro:include filename="$(find src_gazebo)/urdf/src_body.trans" /> -->
+  <link name="base_footprint" />
   <link name="base_link">
     <inertial>
@@ -25,4 +26,9 @@
     </collision>
   </link>
+  <joint name="base_footprint_joint" type="fixed">
+    <parent link="base_footprint"/>
+    <child link="base_link"/>
+    <origin xyz="0 0 0" rpy="0 0 0"/>
+  </joint>
   <link name="lf_steering_hinge_link">
     <inertial>
