Commit message: stick spawn done

File: sensor_stick/urdf/sensor_stick.gazebo.xacro (robot description, xacro)
@@ -66,9 +66,9 @@
       <plugin name="depth_camera_controller" filename="libgazebo_ros_camera.so">
         <!-- Change namespace, camera name and topics so -
-             * Raw images are published to: /custom_ns/custom_camera/custom_image
-             * Depth images are published to: /custom_ns/custom_camera/custom_image_depth
-             * Raw image camera info is published to: /custom_ns/custom_camera/custom_info_raw
-             * Depth image camera info is published to: /custom_ns/custom_camera/custom_info_depth
-             * Point cloud is published to: /custom_ns/custom_camera/custom_points
+             * Raw images are published to /custom_ns/custom_camera/custom_image
+             * Depth images are published to /custom_ns/custom_camera/custom_image_depth
+             * Raw image camera info is published to /custom_ns/custom_camera/custom_info_raw
+             * Depth image camera info is published to /custom_ns/custom_camera/custom_info_depth
+             * Point cloud is published to /custom_ns/custom_camera/custom_points
         -->
         <ros>
@@ -85,5 +85,5 @@
         <!-- <frame_name>custom_frame</frame_name> -->
         <!-- hackbaseline is the length of baseline, its an important parameter for stereo camera. -->
-        <!-- hackbaseline reference : http://docs.ros.org/en/melodic/api/sensor_msgs/html/msg/CameraInfo.html -->
+        <!-- hackbaseline reference  http://docs.ros.org/en/melodic/api/sensor_msgs/html/msg/CameraInfo.html -->
         <!-- <hack_baseline>0.07</hack_baseline> -->
         <!-- No need to repeat distortion parameters or to set autoDistortion -->

File: sensor_stick/urdf/sensor_stick.urdf.xacro (robot description, xacro)
@@ -1,5 +1,4 @@
 <?xml version="1.0"?>
 <robot name="sensor_stick" xmlns:xacro="http://www.ros.org/wiki/xacro">
-  <!--Define constants-->
   <xacro:property name="PI" value="3.14159"/>
   <xacro:property name="mass1" value="10" />
@@ -76,5 +75,5 @@
     <origin xyz="0 0 0" rpy="0 0 0"/>
     <geometry>
-      <mesh filename="package://sensor_stick/meshes/asus_xtion.dae"/>
+      <mesh filename="$(find sensor_stick)/meshes/asus_xtion.dae"/>
     </geometry>
   </visual>
